Commit message: fix bugs

File: mrobot_gazebo/urdf/mrobot_body.urdf.xacro (robot description, xacro)
@@ -2,14 +2,17 @@
 <robot name="mrobot" xmlns:xacro="http://www.ros.org/wiki/xacro">
     <!-- Defining the colors used in this robot -->
-    <material name="Black">
+    <material name="yellow">
+        <color rgba="1 0.4 0 1"/>
+    </material>
+    <material name="black">
         <color rgba="0 0 0 1"/>
     </material>
-    <material name="White">
+    <material name="white">
         <color rgba="1 1 1 1"/>
     </material>
-    <material name="Blue">
+    <material name="blue">
         <color rgba="0 0 1 1"/>
     </material>
-    <material name="Red">
+    <material name="red">
         <color rgba="1 0 0 1"/>
     </material>
@@ -69,5 +72,5 @@
                     <cylinder length="${wheel_height}" radius="${wheel_radius}" />
                 </geometry>
-                <material name="Black" />
+                <material name="black" />
             </visual>
             <collision>
@@ -77,8 +80,8 @@
                 </geometry>
             </collision>
-            <cylinder_inertial_matrix  m="${wheel_mass}" r="${wheel_radius}" h="${wheel_height}" />
+            <xacro:cylinder_inertial_matrix  m="${wheel_mass}" r="${wheel_radius}" h="${wheel_height}" />
         </link>
         <gazebo reference="wheel_${lr}_link">
-            <material>Gazebo/Black</material>
+            <material>Gazebo/black</material>
         </gazebo>
         <joint name="base_to_wheel_${lr}_joint" type="continuous">
@@ -107,5 +110,5 @@
                     <sphere radius="${caster_radius}" />
                 </geometry>
-                <material name="Black" />
+                <material name="black" />
             </visual>
             <collision>
@@ -115,8 +118,8 @@
                 <origin xyz="0 0 0 " rpy="0 0 0" />
             </collision>
-            <sphere_inertial_matrix  m="${caster_mass}" r="${caster_radius}" />
+            <xacro:sphere_inertial_matrix  m="${caster_mass}" r="${caster_radius}" />
         </link>
         <gazebo reference="${fb}_caster_link">
-            <material>Gazebo/Black</material>
+            <material>Gazebo/black</material>
         </gazebo>
         <joint name="base_to_${fb}_caster_joint" type="fixed">
@@ -129,5 +132,5 @@
     <xacro:macro name="plate" params="num parent">
         <link name="plate_${num}_link">
-            <cylinder_inertial_matrix  m="0.1" r="${base_link_radius}" h="${base_link_length}" />
+            <xacro:cylinder_inertial_matrix  m="0.1" r="${base_link_radius}" h="${base_link_length}" />
             <visual>
                 <origin xyz=" 0 0 0 " rpy="0 0 0" />
@@ -204,5 +207,5 @@
         <!--Actual body/chassis of the robot-->
         <link name="base_link">
-            <cylinder_inertial_matrix  m="${base_mass}" r="${base_link_radius}" h="${base_link_length}" />
+            <xacro:cylinder_inertial_matrix  m="${base_mass}" r="${base_link_radius}" h="${base_link_length}" />
             <visual>
                 <origin xyz=" 0 0 0" rpy="0 0 0" />
@@ -223,20 +226,20 @@
         </gazebo>
         <!-- Wheel Definitions -->
-        <wheel lr="right"  translateY="1" />
-        <wheel lr="left"  translateY="-1" />
+        <xacro:wheel lr="right"  translateY="1" />
+        <xacro:wheel lr="left"  translateY="-1" />
         <!-- Casters Definitions -->
-        <caster fb="front"  translateX="-1" />
+        <xacro:caster fb="front"  translateX="-1" />
         <!-- plates and standoff Definitions -->
-        <mrobot_standoff_2in parent="base_link" number="1" x_loc="-${standoff_x/2 + 0.03}" y_loc="-${standoff_y - 0.03}" z_loc="${plate_height/2}"/>
-        <mrobot_standoff_2in parent="base_link" number="2" x_loc="-${standoff_x/2 + 0.03}" y_loc="${standoff_y - 0.03}" z_loc="${plate_height/2}"/>
-        <mrobot_standoff_2in parent="base_link" number="3" x_loc="${standoff_x/2}" y_loc="-${standoff_y}" z_loc="${plate_height/2}"/>
-        <mrobot_standoff_2in parent="base_link" number="4" x_loc="${standoff_x/2}" y_loc="${standoff_y}" z_loc="${plate_height/2}"/>
-        <mrobot_standoff_2in parent="standoff_2in_1_link" number="5" x_loc="0" y_loc="0" z_loc="${plate_height}"/>
-        <mrobot_standoff_2in parent="standoff_2in_2_link" number="6" x_loc="0" y_loc="0" z_loc="${plate_height}"/>
-        <mrobot_standoff_2in parent="standoff_2in_3_link" number="7" x_loc="0" y_loc="0" z_loc="${plate_height}"/>
-        <mrobot_standoff_2in parent="standoff_2in_4_link" number="8" x_loc="0" y_loc="0" z_loc="${plate_height}"/>
+        <xacro:mrobot_standoff_2in parent="base_link" number="1" x_loc="-${standoff_x/2 + 0.03}" y_loc="-${standoff_y - 0.03}" z_loc="${plate_height/2}"/>
+        <xacro:mrobot_standoff_2in parent="base_link" number="2" x_loc="-${standoff_x/2 + 0.03}" y_loc="${standoff_y - 0.03}" z_loc="${plate_height/2}"/>
+        <xacro:mrobot_standoff_2in parent="base_link" number="3" x_loc="${standoff_x/2}" y_loc="-${standoff_y}" z_loc="${plate_height/2}"/>
+        <xacro:mrobot_standoff_2in parent="base_link" number="4" x_loc="${standoff_x/2}" y_loc="${standoff_y}" z_loc="${plate_height/2}"/>
+        <xacro:mrobot_standoff_2in parent="standoff_2in_1_link" number="5" x_loc="0" y_loc="0" z_loc="${plate_height}"/>
+        <xacro:mrobot_standoff_2in parent="standoff_2in_2_link" number="6" x_loc="0" y_loc="0" z_loc="${plate_height}"/>
+        <xacro:mrobot_standoff_2in parent="standoff_2in_3_link" number="7" x_loc="0" y_loc="0" z_loc="${plate_height}"/>
+        <xacro:mrobot_standoff_2in parent="standoff_2in_4_link" number="8" x_loc="0" y_loc="0" z_loc="${plate_height}"/>
         <!-- plate Definitions -->
-        <plate num="1"  parent="base_link" />
-        <plate num="2"  parent="plate_1_link" />
+        <xacro:plate num="1"  parent="base_link" />
+        <xacro:plate num="2"  parent="plate_1_link" />
         <!-- controller -->
         <gazebo>
